Commit message: Updated with ros2 control

File: description/robot.urdf.xacro (robot description, xacro)
@@ -2,5 +2,4 @@
 <robot xmlns:xacro="http://www.ros.org/wiki/xacro"  name="robot">
     <xacro:include filename= "robot_core.xacro" />
-    <!--<xacro:include filename= "gazebo_control.xacro" /> -->
     <xacro:include filename= "lidar.xacro" />
     <xacro:include filename= "camera.xacro" />

File: description/robot_core.xacro (robot description, xacro)
@@ -153,3 +153,23 @@
         <material>Gazebo/Orange</material>
     </gazebo>
+     <transmission name="Left_side_trans">
+      <type>transmission_interface/SimpleTransmission</type>
+      <joint name="front_left_wheel_joint">
+        <hardwareInterface>hardware_interface/EffortJointInterface</hardwareInterface>
+      </joint>
+      <actuator name="back_left_wheel_joint">
+        <hardwareInterface>hardware_interface/EffortJointInterface</hardwareInterface>
+        <mechanicalReduction>1</mechanicalReduction>
+      </actuator>
+    </transmission>
+    <transmission name="Right_side_trans">
+      <type>transmission_interface/SimpleTransmission</type>
+      <joint name="front_right_wheel_joint">
+        <hardwareInterface>hardware_interface/EffortJointInterface</hardwareInterface>
+      </joint>
+      <actuator name="back_right_wheel_joint">
+        <hardwareInterface>hardware_interface/EffortJointInterface</hardwareInterface>
+        <mechanicalReduction>1</mechanicalReduction>
+      </actuator>
+    </transmission>
 </robot>

File: description/ros2_control.xacro (robot description, xacro)
@@ -7,5 +7,5 @@
         <joint name = "back_left_wheel_joint">
             <command_interface name="velocity">
-                <param name = "min">10</param>
+                <param name = "min">-10</param>
                 <param name = "max">10</param>
             </command_interface>
@@ -15,5 +15,5 @@
         <joint name = "back_right_wheel_joint">
             <command_interface name="velocity">
-                <param name = "min">10</param>
+                <param name = "min">-10</param>
                 <param name = "max">10</param>
             </command_interface>
