Commit message: Added simulated gazebo camera

File: description/camera.xacro (robot description, xacro)
@@ -9,5 +9,5 @@
         <visual>
             <geometry>
-                <box size = "0.010 0.0255 0.255"/>
+                <box size = "0.010 0.0255 0.0255"/>
             </geometry>
             <material name = "red" />
@@ -22,32 +22,24 @@
     <gazebo reference = "camera_link">
         <material>Gazebo/White</material>
-<!--
-        <sensor name = "laser" type = "ray">
+        <sensor name = "camera" type = "camera">
             <pose> 0 0 0 0 0 0 </pose>
             <visualize>true</visualize>
             <update_rate>10</update_rate>
-            <ray>
-                <scan>
-                    <horizontal>
-                        <samples>360</samples>
-                        <resolution>1</resolution>
-                        <min_angle>-3.14</min_angle>
-                        <max_angle>3.14</max_angle>
-                    </horizontal>
-                </scan>
-                <range>
-                    <min>0.3</min>
-                    <max>12</max>
-                    <resolution>0.01</resolution>
-                </range>
-            </ray>
-            <plugin name = "laser_controller" filename = "libgazebo_ros_ray_sensor.so">
-                <ros>
-                    <argument>~/out:=scan</argument>
-                </ros>
-                <output_type>sensor_msgs/laserScan</output_type>
-                <frame_name>laser_frame</frame_name>
+            <camera>
+                <horizontal_fov>1.089</horizontal_fov>
+                <image>
+                    <format>R8G8B8</format>
+                    <width>640</width>
+                    <height>480</height>
+                </image>
+                <clip>
+                    <near>0.05</near>
+                    <far>8.0</far>
+                </clip>
+            </camera>
+            <plugin name = "camera_controller" filename = "libgazebo_ros_camera.so">
+                <frame_name>camera_link_optical</frame_name>
             </plugin>
-        </sensor> -->
+        </sensor>
     </gazebo>
 </robot>

Commit message: Added controllers, Additional robot description

File: description/camera.xacro (robot description, xacro)
@@ -39,4 +39,5 @@
             </camera>
             <plugin name = "camera_controller" filename = "libgazebo_ros_camera.so">
+                <imageTopicName>image_raw</imageTopicName>
                 <frame_name>camera_link_optical</frame_name>
             </plugin>

File: description/lidar.xacro (robot description, xacro)
@@ -4,10 +4,10 @@
         <parent link = "chassis"/>
         <child link = "laser_frame"/>
-        <origin xyz = "0.1795 0.046 0.055" rpy = "0 0 0"/>
+        <origin xyz = "0.1795 0.046 0.07" rpy = "0 0 0"/>
     </joint>
     <link name ="laser_frame">
         <visual>
             <geometry>
-                <cylinder radius = "0.035" length ="0.055"/>
+                <cylinder radius = "0.035" length ="0.07"/>
             </geometry>
             <material name = "orange" />
@@ -24,4 +24,5 @@
     </link>
     <gazebo reference = "laser_frame">
+        <material>Gazebo/White</material>
         <sensor name = "laser" type = "ray">
             <pose> 0 0 0 0 0 0 </pose>
@@ -32,5 +33,4 @@
                     <horizontal>
                         <samples>360</samples>
-                        <resolution>1</resolution>
                         <min_angle>-3.14</min_angle>
                         <max_angle>3.14</max_angle>
@@ -40,5 +40,4 @@
                     <min>0.3</min>
                     <max>12</max>
-                    <resolution>0.01</resolution>
                 </range>
             </ray>
@@ -47,9 +46,8 @@
                     <argument>~/out:=scan</argument>
                 </ros>
-                <output_type>sensor_msgs/laserScan</output_type>
+                <output_type>sensor_msgs/LaserScan</output_type>
                 <frame_name>laser_frame</frame_name>
             </plugin>
         </sensor>
-        <material>Gazebo/White</material>
     </gazebo>
 </robot>

File: description/robot_core.xacro (robot description, xacro)
@@ -17,4 +17,12 @@
     <link name = "base_link">
     </link>
+    <!-- BASE FOOTPRINT LINK-->
+    <joint name = "base_footprint_joint" type = "fixed">
+        <parent link = "base_link"/>
+        <child link = "base_footprint"/>
+        <origin xyz ="0 0 0" rpy="0 0 0"/>
+    </joint>
+    <link name = "base_footprint">
+    </link>
     <!-- CHASSIS LINK -->
     <joint name = "chassis_joint" type = "fixed">
@@ -46,5 +54,5 @@
     </gazebo>
     <!-- LEFT WHEEL REAR -->
-    <joint name = "back_left_wheel_joint" type = "continuous">
+    <joint name = "back_left_wheel_joint" type = "fixed">
         <parent link = "base_link"/>
         <child link = "left_wheel_rear"/>
@@ -59,19 +67,21 @@
             <material name = "blue" />
         </visual>
-        <collision>
-            <geometry>
-                <cylinder radius = "0.06" length ="0.069"/>
-            </geometry>
-            <material name = "blue" />
-        </collision>
-        <xacro:inertial_cylinder mass = "0.1" length = "0.069" radius = "0.06">
-            <origin xyz = "0 0 0" rpy ="0 0 0"/>
-        </xacro:inertial_cylinder>
+        <!-- <collision>
+            <geometry>
+                <cylinder radius = "0.06" length ="0.069"/>
+            </geometry>
+            <material name = "blue" />
+        </collision>
+        <xacro:inertial_cylinder mass = "0.1" length = "0.069" radius = "0.06">
+            <origin xyz = "0 0 0" rpy ="0 0 0"/>
+        </xacro:inertial_cylinder> -->
     </link>
     <gazebo reference = "left_wheel_rear">
         <material>Gazebo/Blue</material>
+        <mu1 value="0.001"/>
+        <mu2 value="0.001"/>
     </gazebo>
     <!-- LEFT WHEEL FRONT-->
-    <joint name = "front_left_wheel_joint" type = "continuous">
+    <joint name = "front_left_wheel_joint" type = "fixed">
         <parent link = "base_link"/>
         <child link = "left_wheel_front"/>
@@ -86,19 +96,48 @@
             <material name = "blue" />
         </visual>
-        <collision>
-            <geometry>
-                <cylinder radius = "0.06" length ="0.069"/>
-            </geometry>
-            <material name = "blue" />
-        </collision>
-        <xacro:inertial_cylinder mass = "0.1" length = "0.069" radius = "0.06">
-            <origin xyz = "0 0 0" rpy ="0 0 0"/>
-        </xacro:inertial_cylinder>
+        <!-- <collision>
+            <geometry>
+                <cylinder radius = "0.06" length ="0.069"/>
+            </geometry>
+            <material name = "blue" />
+        </collision>
+        <xacro:inertial_cylinder mass = "0.1" length = "0.069" radius = "0.06">
+            <origin xyz = "0 0 0" rpy ="0 0 0"/>
+        </xacro:inertial_cylinder> -->
     </link>
     <gazebo reference = "left_wheel_front">
         <material>Gazebo/Blue</material>
+        <mu1 value="0.001"/>
+        <mu2 value="0.001"/>
+    </gazebo>
+    <!-- LEFT DRIVE WHEEL -->
+      <joint name = "left_drive_joint" type = "continuous">
+        <parent link = "base_link"/>
+        <child link = "left_wheel_drive"/>
+        <origin xyz = "0 0.1425 0" rpy="-${pi/2} 0 0"/>
+        <axis xyz = "0 0 1"/>
+    </joint>
+    <link name = "left_wheel_drive">
+        <visual>
+            <geometry>
+                <cylinder radius = "0.06" length ="0.069"/>
+            </geometry>
+            <material name = "blue" />
+        </visual>
+        <collision>
+            <geometry>
+                <cylinder radius = "0.06" length ="0.069"/>
+            </geometry>
+            <material name = "blue" />
+        </collision>
+        <xacro:inertial_cylinder mass = "0.1" length = "0.069" radius = "0.06">
+            <origin xyz = "0 0 0" rpy ="0 0 0"/>
+        </xacro:inertial_cylinder>
+    </link>
+    <gazebo reference = "left_wheel_drive">
+        <material>Gazebo/GreyTransparent</material>
     </gazebo>
      <!-- RIGHTWHEEL REAR -->
-    <joint name = "back_right_wheel_joint" type = "continuous">
+    <joint name = "back_right_wheel_joint" type = "fixed">
         <parent link = "base_link"/>
         <child link = "right_wheel_rear"/>
@@ -113,19 +152,21 @@
             <material name = "orange" />
         </visual>
-        <collision>
-            <geometry>
-                <cylinder radius = "0.06" length ="0.069"/>
-            </geometry>
-            <material name = "orange" />
-        </collision>
-        <xacro:inertial_cylinder mass = "0.1" length = "0.069" radius = "0.06">
-            <origin xyz = "0 0 0" rpy ="0 0 0"/>
-        </xacro:inertial_cylinder>
+        <!-- <collision>
+            <geometry>
+                <cylinder radius = "0.06" length ="0.069"/>
+            </geometry>
+            <material name = "orange" />
+        </collision>
+        <xacro:inertial_cylinder mass = "0.1" length = "0.069" radius = "0.06">
+            <origin xyz = "0 0 0" rpy ="0 0 0"/>
+        </xacro:inertial_cylinder> -->
     </link>
     <gazebo reference = "right_wheel_rear">
         <material>Gazebo/Orange</material>
+        <mu1 value="0.001"/>
+        <mu2 value="0.001"/>
     </gazebo>
      <!-- RIGHTWHEEL FRONT-->
-    <joint name = "front_right_wheel_joint" type = "continuous">
+    <joint name = "front_right_wheel_joint" type = "fixed">
         <parent link = "base_link"/>
         <child link = "right_wheel_front"/>
@@ -140,36 +181,99 @@
             <material name = "orange" />
         </visual>
-        <collision>
-            <geometry>
-                <cylinder radius = "0.06" length ="0.069"/>
-            </geometry>
-            <material name = "orange" />
-        </collision>
-        <xacro:inertial_cylinder mass = "0.1" length = "0.069" radius = "0.06">
-            <origin xyz = "0 0 0" rpy ="0 0 0"/>
-        </xacro:inertial_cylinder>
+        <!-- <collision>
+            <geometry>
+                <cylinder radius = "0.06" length ="0.069"/>
+            </geometry>
+            <material name = "orange" />
+        </collision>
+        <xacro:inertial_cylinder mass = "0.1" length = "0.069" radius = "0.06">
+            <origin xyz = "0 0 0" rpy ="0 0 0"/>
+        </xacro:inertial_cylinder> -->
     </link>
     <gazebo reference = "right_wheel_front">
         <material>Gazebo/Orange</material>
-    </gazebo>
-     <transmission name="Left_side_trans">
-      <type>transmission_interface/SimpleTransmission</type>
-      <joint name="front_left_wheel_joint">
-        <hardwareInterface>hardware_interface/EffortJointInterface</hardwareInterface>
-      </joint>
-      <actuator name="back_left_wheel_joint">
-        <hardwareInterface>hardware_interface/EffortJointInterface</hardwareInterface>
-        <mechanicalReduction>1</mechanicalReduction>
-      </actuator>
-    </transmission>
-    <transmission name="Right_side_trans">
-      <type>transmission_interface/SimpleTransmission</type>
-      <joint name="front_right_wheel_joint">
-        <hardwareInterface>hardware_interface/EffortJointInterface</hardwareInterface>
-      </joint>
-      <actuator name="back_right_wheel_joint">
-        <hardwareInterface>hardware_interface/EffortJointInterface</hardwareInterface>
-        <mechanicalReduction>1</mechanicalReduction>
-      </actuator>
-    </transmission>
+        <mu1 value="0.001"/>
+        <mu2 value="0.001"/>
+    </gazebo>
+    <!-- RIGHT WHEEL DRIVE -->
+     <joint name = "right_drive_joint" type = "continuous">
+        <parent link = "base_link"/>
+        <child link = "right_wheel_drive"/>
+        <origin xyz = "0 -0.1425 0" rpy="${pi/2} 0 0"/>
+        <axis xyz = "0 0 -1"/>
+    </joint>
+    <link name = "right_wheel_drive">
+        <visual>
+            <geometry>
+                <cylinder radius = "0.06" length ="0.069"/>
+            </geometry>
+            <material name = "orange" />
+        </visual>
+        <collision>
+            <geometry>
+                <cylinder radius = "0.06" length ="0.069"/>
+            </geometry>
+            <material name = "orange" />
+        </collision>
+        <xacro:inertial_cylinder mass = "0.1" length = "0.069" radius = "0.06">
+            <origin xyz = "0 0 0" rpy ="0 0 0"/>
+        </xacro:inertial_cylinder>
+    </link>
+    <gazebo reference = "right_wheel_drive">
+        <material>Gazebo/GreyTransparent</material>
+    </gazebo>
+    <!--FRONT BALANCE-->
+    <joint name="front_caster_wheel_joint" type="fixed">
+        <parent link="chassis"/>
+        <child link="caster_wheel_front"/>
+        <origin xyz="0.0975 0 -0.0425"/>
+    </joint>
+    <link name="caster_wheel_front">
+        <visual>
+            <geometry>
+                <sphere radius="0.01475"/>
+            </geometry>
+            <material name="white"/>
+        </visual>
+        <collision>
+            <geometry>
+                <sphere radius="0.01475"/>
+            </geometry>
+        </collision>
+        <xacro:inertial_sphere mass="0.1" radius="0.01475">
+            <origin xyz="0 0 0" rpy="0 0 0"/>
+        </xacro:inertial_sphere>
+    </link>
+    <gazebo reference = "caster_wheel_front">
+        <material>Gazebo/GreyTransparent</material>
+        <mu1 value="0.001"/>
+        <mu2 value="0.001"/>
+    </gazebo>
+    <!-- BACK BALANCE -->
+     <joint name="back_caster_wheel_joint" type="fixed">
+        <parent link="chassis"/>
+        <child link="caster_wheel_back"/>
+        <origin xyz="-0.0975 0 -0.0425"/>
+    </joint>
+    <link name="caster_wheel_back">
+        <visual>
+            <geometry>
+                <sphere radius="0.01475"/>
+            </geometry>
+            <material name="white"/>
+        </visual>
+        <collision>
+            <geometry>
+                <sphere radius="0.01475"/>
+            </geometry>
+        </collision>
+        <xacro:inertial_sphere mass="0.1" radius="0.01475">
+            <origin xyz="0 0 0" rpy="0 0 0"/>
+        </xacro:inertial_sphere>
+    </link>
+    <gazebo reference = "caster_wheel_back">
+        <material>Gazebo/GreyTransparent</material>
+        <mu1 value="0.001"/>
+        <mu2 value="0.001"/>
+    </gazebo>
 </robot>

File: description/ros2_control.xacro (robot description, xacro)
@@ -1,9 +1,9 @@
 <?xml version="1.0"?>
 <robot xmlns:xacro="http://www.ros.org/wiki/xacro">
-    <!-- <ros2_control name = "GazeboSystem" type = "system">
+    <ros2_control name = "GazeboSystem" type = "system">
         <hardware>
             <plugin>gazebo_ros2_control/GazeboSystem</plugin>
         </hardware>
-        <joint name = "back_left_wheel_joint">
+        <joint name = "left_drive_joint">
             <command_interface name="velocity">
                 <param name = "min">-10</param>
@@ -13,5 +13,5 @@
             <state_interface name ="position"/>
         </joint>
-        <joint name = "back_right_wheel_joint">
+        <joint name = "right_drive_joint">
             <command_interface name="velocity">
                 <param name = "min">-10</param>
@@ -21,7 +21,7 @@
             <state_interface name ="position"/>
         </joint>
-    </ros2_control> -->
+    </ros2_control>
     <!-- CHANGE NUMBERS AS PROJECT DEVELOPS -->
-    <ros2_control name = "RealRobot" type = "system">
+    <!-- <ros2_control name = "RealRobot" type = "system">
         <hardware>
             <plugin>diffdrive_arduino/DiffDriveArduino</plugin>
@@ -50,5 +50,5 @@
             <state_interface name ="position"/>
         </joint>
-    </ros2_control>
+    </ros2_control> -->
     <gazebo>
         <plugin name="gazebo_ros2_control" filename="libgazebo_ros2_control.so">
