Commit message: lidar link rotation to match real robot

File: description/lidar.xacro (robot description, xacro)
@@ -20,5 +20,5 @@
         </collision>
         <xacro:inertial_cylinder mass = "0.1" length = "0.055" radius = "0.035">
-            <origin xyz = "0 0 0" rpy ="0 0 0"/>
+            <origin xyz = "0 0 0" rpy ="0 0 ${pi}"/>
         </xacro:inertial_cylinder>
     </link>

Commit message: fixing lidar transform

File: description/lidar.xacro (robot description, xacro)
@@ -4,5 +4,5 @@
         <parent link = "chassis"/>
         <child link = "laser_frame"/>
-        <origin xyz = "0.1795 0.046 0.07" rpy = "0 0 0"/>
+        <origin xyz = "0.1795 0.046 0.07" rpy = "0 0 ${pi}"/>
     </joint>
     <link name ="laser_frame">
@@ -20,5 +20,5 @@
         </collision>
         <xacro:inertial_cylinder mass = "0.1" length = "0.055" radius = "0.035">
-            <origin xyz = "0 0 0" rpy ="0 0 ${pi}"/>
+            <origin xyz = "0 0 0" rpy ="0 0 0"/>
         </xacro:inertial_cylinder>
     </link>
