Commit message: Update to robot core

File: description/robot_core.xacro (robot description, xacro)
@@ -14,9 +14,6 @@
         <color rgba="0 0 0 1" />
     </material>
-    <!-- BASE LINK -->
-    <link name = "base_link">
-    </link>
     <!-- BASE FOOTPRINT LINK-->
-    <joint name = "base_footprint_joint" type = "fixed">
+    <joint name = "base_link_joint" type = "fixed">
         <parent link = "base_link"/>
         <child link = "base_footprint"/>
@@ -25,5 +22,12 @@
     <link name = "base_footprint">
     </link>
-    <!-- CHASSIS LINK -->
+    <!-- BASE LINK -->
+    <!-- <joint name = "base_link_joint" type = "fixed">
+        <parent link = "base_footprint"/>
+        <child link = "base_link"/>
+        <origin xyz ="0 0 0" rpy="0 0 0"/>
+    </joint> -->
+    <link name = "base_link">
+    </link>
     <joint name = "chassis_joint" type = "fixed">
         <parent link = "base_link"/>

Commit message: fix for base_link odom connection

File: description/robot_core.xacro (robot description, xacro)
@@ -14,18 +14,4 @@
         <color rgba="0 0 0 1" />
     </material>
-    <!-- BASE FOOTPRINT LINK-->
-    <joint name = "base_link_joint" type = "fixed">
-        <parent link = "base_link"/>
-        <child link = "base_footprint"/>
-        <origin xyz ="0 0 0" rpy="0 0 0"/>
-    </joint>
-    <link name = "base_footprint">
-    </link>
-    <!-- BASE LINK -->
-    <!-- <joint name = "base_link_joint" type = "fixed">
-        <parent link = "base_footprint"/>
-        <child link = "base_link"/>
-        <origin xyz ="0 0 0" rpy="0 0 0"/>
-    </joint> -->
     <link name = "base_link">
     </link>

Commit message: joystick with mapping functionality

File: description/robot_core.xacro (robot description, xacro)
@@ -16,4 +16,12 @@
     <link name = "base_link">
     </link>
+    <!-- BASE_FOOTPRINT LINK -->
+    <joint name="base_footprint_joint" type="fixed">
+        <parent link="base_link"/>
+        <child link="base_footprint"/>
+        <origin xyz="0 0 0" rpy="0 0 0"/>
+    </joint>
+    <link name="base_footprint">
+    </link>
     <joint name = "chassis_joint" type = "fixed">
         <parent link = "base_link"/>

Commit message: remove base footprint

File: description/robot_core.xacro (robot description, xacro)
@@ -17,5 +17,5 @@
     </link>
     <!-- BASE_FOOTPRINT LINK -->
-    <joint name="base_footprint_joint" type="fixed">
+    <!-- <joint name="base_footprint_joint" type="fixed">
         <parent link="base_link"/>
         <child link="base_footprint"/>
@@ -23,5 +23,5 @@
     </joint>
     <link name="base_footprint">
-    </link>
+    </link> -->
     <joint name = "chassis_joint" type = "fixed">
         <parent link = "base_link"/>

Commit message: base footprint added back

File: description/robot_core.xacro (robot description, xacro)
@@ -17,5 +17,5 @@
     </link>
     <!-- BASE_FOOTPRINT LINK -->
-    <!-- <joint name="base_footprint_joint" type="fixed">
+    <joint name="base_footprint_joint" type="fixed">
         <parent link="base_link"/>
         <child link="base_footprint"/>
@@ -23,5 +23,5 @@
     </joint>
     <link name="base_footprint">
-    </link> -->
+    </link>
     <joint name = "chassis_joint" type = "fixed">
         <parent link = "base_link"/>
